File: Flachbaugruppe.kicad_pcb (KiCad board)
At the start: 4 copper layers, 154 x 98.5 mm, 51 parts, among them J1 Input A, J2 Input B, J3 Outout, J4 GND, SW2 SW_SP3T_NR01103, U1 LM7818_TO220, U2 4013, U3 LM555xM, U4 LM7805_TO220, U5 LM358, U6 ATmega328P-P, Y1 16 MHz

Commit message: Update
Parts:
- moved C16 1.00 mm to (160.1, 152.5)
- turned R10 to 180 degrees
Routing:
- net Net-(U2A-Q): track 21.6 -> 125.7 mm, vias 0 -> 1
- net Net-(DS1-D7): track 0.00 -> 93.7 mm, vias 0 -> 1
- net Net-(DS1-D6): track 0.00 -> 90.3 mm, vias 0 -> 1
- net Net-(DS1-D5): track 0.00 -> 78.9 mm, vias 0 -> 1
- net Net-(DS1-D4): track 0.00 -> 66.6 mm, vias 0 -> 2
- net Net-(DS1-E): track 0.00 -> 61.2 mm, vias 0 -> 2
- net Net-(J3-Pin_1): track 63.8 -> 115.5 mm
- net Net-(DS1-RS): track 0.00 -> 50.7 mm
- net +5V: track 3.62 -> 45.3 mm, vias 1 -> 2
- net Net-(DS1-VO): track 0.00 -> 36.9 mm
- net Net-(U6-XTAL2/PB7): track 0.00 -> 33.2 mm, vias 0 -> 1
- net Net-(U6-PB0): track 0.00 -> 33.1 mm
- net GND: track 58.7 -> 86.8 mm, vias 10 -> 18
- net Net-(U6-PC0): track 0.00 -> 17.2 mm, vias 0 -> 1
- net Net-(U5A--): track 4.26 -> 15.5 mm
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
Commit message: Finalize PCB design, Gerber files and manufacturing documentation
Parts:
- renumbered REF** to H1, REF** to H2, REF** to H3, REF** to H4
Routing:
- net Net-(U6-XTAL2/PB7): track 33.2 -> 33.9 mm
