File: Flachbaugruppe.kicad_sch (KiCad schematic)
At the start: 47 parts, among them J1 Input A, J2 Input B, J3 Outout, J4 GND, SW2 SW_SP3T_NR01103, U1 LM7818_TO220, U2 4013, U3 LM555xM, U4 LM7805_TO220, U5 LM358, U6 ATmega328P-P, Y1 16 MHz

Commit message: Finalize PCB design, Gerber files and manufacturing documentation
Parts:
- C5, C7: symbol Device:C -> Device:C_Polarized
Changed lines of the file:
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@@
 	)
 	(symbol
-		(lib_id "Device:C")
+		(lib_id "Device:C_Polarized")
 		(at 162.56 99.06 0)
 		(unit 1)
@@
 		(fields_autoplaced yes)
 		(property "Reference" "C5"
-			(at 166.37 97.7899 0)
+			(at 166.37 96.9009 0)
 			(effects
 				(font
@@
 		)
 		(property "Value" "33uf"
-			(at 166.37 100.3299 0)
+			(at 166.37 99.4409 0)
 			(effects
 				(font
@@
 			)
 		)
-		(property "Description" "Unpolarized capacitor"
+		(property "Description" "Polarized capacitor"
 			(at 162.56 99.06 0)
 			(effects
@@
 	)
 	(symbol
-		(lib_id "Device:C")
+		(lib_id "Device:C_Polarized")
 		(at 147.32 99.06 0)
 		(unit 1)
@@
 		(fields_autoplaced yes)
 		(property "Reference" "C7"
-			(at 151.13 97.7899 0)
+			(at 151.13 96.9009 0)
 			(effects
 				(font
@@
 		)
 		(property "Value" "3,3uf"
-			(at 151.13 100.3299 0)
+			(at 151.13 99.4409 0)
 			(effects
 				(font
@@
 			)
 		)
-		(property "Description" "Unpolarized capacitor"
+		(property "Description" "Polarized capacitor"
 			(at 147.32 99.06 0)
 			(effects
